Commit message: 电机驱动框架代码

File: pca9685_ros2_control_example/description/description.urdf.xacro (robot description, xacro)
@@ -5,25 +5,21 @@
       <plugin>pca9685_hardware_interface/Pca9685SystemHardware</plugin>
     </hardware>
-    <joint name="joint_0">
-      <command_interface name="velocity"/>
-      <state_interface name="velocity"/>
-    </joint>
     <joint name="joint_1">
+      <param name="channel">0</param>
       <command_interface name="velocity"/>
       <state_interface name="velocity"/>
     </joint>
     <joint name="joint_2">
+      <param name="channel">1</param>
       <command_interface name="velocity"/>
       <state_interface name="velocity"/>
     </joint>
     <joint name="joint_3">
+      <param name="channel">2</param>
       <command_interface name="velocity"/>
       <state_interface name="velocity"/>
     </joint>
     <joint name="joint_4">
-      <command_interface name="velocity"/>
-      <state_interface name="velocity"/>
-    </joint>
-    <joint name="joint_5">
+      <param name="channel">3</param>
       <command_interface name="velocity"/>
       <state_interface name="velocity"/>
